Commit message: Update sam_bot_description.urdf
Fix inertia setting for chassis(base_link) and wheels, as well as the negative radius of caster(front_caster link).

File: sam_bot_description/src/description/sam_bot_description.urdf (robot description, URDF)
Before this commit: robot sam_bot, 3 links, 2 joints
Links:
- link front_caster: geometry collision sphere radius=${(wheel_radius+wheel_zoff-(base_height/2))}; visual sphere radius=${(wheel_radius+wheel_zoff-(base_height/2))}

Commit message: Update sam_bot for sensor tutorials

File: sam_bot_description/src/description/sam_bot_description.urdf (robot description, URDF)
Before this commit: robot sam_bot, 4 links, 3 joints
Links:
- added link camera_depth_frame
- added link camera_link, mass 0.035; collision box size=0.015 0.130 0.022; visual box size=0.015 0.130 0.022
- added link lidar_link, mass 0.125; collision cylinder length=0.055 radius=0.0508; visual cylinder length=0.055 radius=0.0508
Joints:
- added joint camera_depth_joint: type fixed, parent camera_link, child camera_depth_frame, origin xyz=0 0 0 rpy=${-pi/2} 0 ${-pi}
- added joint camera_joint: type fixed, parent base_link, child camera_link, origin xyz=0.215 0 0.05 rpy=0 0 0
- added joint lidar_joint: type fixed, parent base_link, child lidar_link, origin xyz=0 0 0.12 rpy=0 0 0

Commit message: Edit URDF to fix frame referenced by camera plugin

File: sam_bot_description/src/description/sam_bot_description.urdf (robot description, URDF)
Before this commit: robot sam_bot, 7 links, 6 joints
Joints:
- joint camera_depth_joint: origin xyz=0 0 0 rpy=${-pi/2} 0 ${-pi} -> xyz=0 0 0 rpy=${-pi/2} 0 ${-pi/2}
