Commit message: Update turtlebot urdf

File: nav2_gps_waypoint_follower_demo/urdf/turtlebot3_waffle_gps.urdf (robot description, URDF)
Before this commit: robot turtlebot3_waffle, 14 links, 13 joints
Joints:
- joint base_joint: child base_link -> base_footprint; origin xyz=0 0 0.010 rpy=0 0 0 -> xyz=0 0 -0.010 rpy=0 0 0; parent base_footprint -> base_link
